File: skedd-jtag6.kicad_pcb (KiCad board)
At the start: 2 copper layers, 11.4 x 16.5 mm, 2 parts, among them J1 Conn_02x03_Odd_Even, J2 Conn_01x06

Commit message: Tweaks.
Parts:
- moved J1 2.54 mm to (124.5, 76.2)
- moved J2 2.54 mm to (130.8, 82.5)
Routing:
- net GND: track 17.9 -> 9.48 mm
- net /TCK: track 5.34 -> 8.29 mm
- net /TDO: track 7.82 -> 6.92 mm
